File: MainBoardTrans_Unlimited2026/MainBoardTrans_Unlimited2026.kicad_pcb (KiCad board)
At the start: 2 copper layers, 100 x 90 mm, 65 parts, among them J10 DSN-MINI-360, J11 pin_H, J12 RST, J13 I2C, J14 RJ45_Shielded, J15 Solenoid, J6 molex, J7 xt30, J8 Tblock, J9 ID-BAT, Q1 IRFZ44N, U1 TA6586, U10 TA6586, U2 TA6586, U3 TA6586, U4 TA6586, U5 TA6586, U6 ESP32-S3-DEVKITC-1, U7 ACS712xLCTR-05B, U8 BNO085, U9 AMS1117-3.3

Commit message: update pcb
Parts:
- renumbered J1 to M1, J2 to M2, J3 to M3, J4 to M4, J5 to M5, J16 to M6
Connections:
- net Net-(J15-Pin_2) renamed Selonoid
- net Net-(J16-Pin_1) renamed FO6
- net Net-(J16-Pin_2) renamed BO6
Changed lines of the file:
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@@
 			)
 		)
+		(model "${KICAD10_3DMODEL_DIR}/Connector_RJ.3dshapes/RJ45_Amphenol_RJHSE538X.step"
+			(offset
+				(xyz 0 0 0)
+			)
+			(scale
+				(xyz 1 1 1)
+			)
+			(rotate
+				(xyz 0 0 0)
+			)
+		)
 	)
 	(footprint "Fuse:Fuse_Bourns_MF-RHT300"
@@
 		(descr "terminal block MaiXu MX126-5.0-02P, 2 pins, pitch 5mm, size 10.5x7.8mm, drill diameter 1.3mm, pad diameter 2.8mm, https://www.lcsc.com/datasheet/lcsc_datasheet_2309150913_MAX-MX126-5-0-03P-GN01-Cu-S-A_C5188435.pdf")
 		(tags "THT terminal block MaiXu MX126-5.0-02P pitch 5mm size 10.5x7.8mm drill 1.3mm pad 2.8mm")
-		(property "Reference" "J16"
+		(property "Reference" "M6"
 			(at 2.25 -5.12 90)
 			(layer "F.SilkS")
@@
 			(remove_unused_layers no)
 			(roundrect_rratio 0.089286)
-			(net "Net-(J16-Pin_1)")
+			(net "FO6")
 			(pinfunction "Pin_1_1")
 			(pintype "passive")
@@
 			(layers "*.Cu" "*.Mask")
 			(remove_unused_layers no)
-			(net "Net-(J16-Pin_2)")
+			(net "BO6")
 			(pinfunction "Pin_2_2")
 			(pintype "passive")
@@
 			)
 		)
+		(model "${KICAD10_3DMODEL_DIR}/TerminalBlock_Phoenix.3dshapes/TerminalBlock_Phoenix_MKDS-1,5-2_1x02_P5.00mm_Horizontal.step"
+			(offset
+				(xyz 0 0 0)
+			)
+			(scale
+				(xyz 1 1 1)
+			)
+			(rotate
+				(xyz 0 0 0)
+			)
+		)
 	)
 	(footprint "Capacitor_THT:CP_Radial_D10.0mm_P5.00mm"
@@
 		(descr "terminal block MaiXu MX126-5.0-02P, 2 pins, pitch 5mm, size 10.5x7.8mm, drill diameter 1.3mm, pad diameter 2.8mm, https://www.lcsc.com/datasheet/lcsc_datasheet_2309150913_MAX-MX126-5-0-03P-GN01-Cu-S-A_C5188435.pdf")
 		(tags "THT terminal block MaiXu MX126-5.0-02P pitch 5mm size 10.5x7.8mm drill 1.3mm pad 2.8mm")
-		(property "Reference" "J3"
+		(property "Reference" "M3"
 			(at 2.25 -5.12 90)
 			(layer "F.SilkS")
@@
 		)
 		(embedded_fonts no)
-		(model "${KICAD10_3DMODEL_DIR}/TerminalBlock.3dshapes/TerminalBlock_MaiXu_MX126-5.0-02P_1x02_P5.00mm.step"
+		(model "${KICAD10_3DMODEL_DIR}/TerminalBlock_Phoenix.3dshapes/TerminalBlock_Phoenix_MKDS-1,5-2_1x02_P5.00mm_Horizontal.step"
 			(offset
 				(xyz 0 0 0)
@@
 		(descr "terminal block MaiXu MX126-5.0-02P, 2 pins, pitch 5mm, size 10.5x7.8mm, drill diameter 1.3mm, pad diameter 2.8mm, https://www.lcsc.com/datasheet/lcsc_datasheet_2309150913_MAX-MX126-5-0-03P-GN01-Cu-S-A_C5188435.pdf")
 		(tags "THT terminal block MaiXu MX126-5.0-02P pitch 5mm size 10.5x7.8mm drill 1.3mm pad 2.8mm")
-		(property "Reference" "J2"
+		(property "Reference" "M2"
 			(at 2.25 -5.12 90)
 			(layer "F.SilkS")
@@
 		)
 		(embedded_fonts no)
-		(model "${KICAD10_3DMODEL_DIR}/TerminalBlock.3dshapes/TerminalBlock_MaiXu_MX126-5.0-02P_1x02_P5.00mm.step"
+		(model "${KICAD10_3DMODEL_DIR}/TerminalBlock_Phoenix.3dshapes/TerminalBlock_Phoenix_MKDS-1,5-2_1x02_P5.00mm_Horizontal.step"
 			(offset
 				(xyz 0 0 0)
@@
 			(layers "*.Cu" "*.Mask")
 			(remove_unused_layers no)
-			(net "Net-(J15-Pin_2)")
+			(net "Selonoid")
 			(pinfunction "Pin_2_2")
 			(pintype "passive")
@@
 		)
 		(embedded_fonts no)
-		(model "${KICAD10_3DMODEL_DIR}/TerminalBlock.3dshapes/TerminalBlock_MaiXu_MX126-5.0-02P_1x02_P5.00mm.step"
+		(model "${KICAD10_3DMODEL_DIR}/TerminalBlock_Phoenix.3dshapes/TerminalBlock_Phoenix_MKDS-1,5-2_1x02_P5.00mm_Horizontal.step"
 			(offset
 				(xyz 0 0 0)
@@
 			(layers "*.Cu" "*.Mask")
 			(remove_unused_layers no)
-			(net "Net-(J16-Pin_2)")
+			(net "BO6")
 			(pinfunction "BO1_BO1")
 			(pintype "bidirectional")
@@
 			(layers "*.Cu" "*.Mask")
 			(remove_unused_layers no)
-			(net "Net-(J16-Pin_2)")
+			(net "BO6")
 			(pinfunction "BO2_BO2")
 			(pintype "bidirectional")
@@
 			(layers "*.Cu" "*.Mask")
 			(remove_unused_layers no)
-			(net "Net-(J16-Pin_1)")
+			(net "FO6")
 			(pinfunction "FO1_FO1")
 			(pintype "bidirectional")
@@
 			(layers "*.Cu" "*.Mask")
 			(remove_unused_layers no)
-			(net "Net-(J16-Pin_1)")
+			(net "FO6")
 			(pinfunction "FO2_FO2")
 			(pintype "bidirectional")
@@
 		(descr "terminal block MaiXu MX126-5.0-02P, 2 pins, pitch 5mm, size 10.5x7.8mm, drill diameter 1.3mm, pad diameter 2.8mm, https://www.lcsc.com/datasheet/lcsc_datasheet_2309150913_MAX-MX126-5-0-03P-GN01-Cu-S-A_C5188435.pdf")
 		(tags "THT terminal block MaiXu MX126-5.0-02P pitch 5mm size 10.5x7.8mm drill 1.3mm pad 2.8mm")
-		(property "Reference" "J4"
+		(property "Reference" "M4"
 			(at 2.25 -5.12 90)
 			(layer "F.SilkS")
@@
 		)
 		(embedded_fonts no)
-		(model "${KICAD10_3DMODEL_DIR}/TerminalBlock.3dshapes/TerminalBlock_MaiXu_MX126-5.0-02P_1x02_P5.00mm.step"
+		(model "${KICAD10_3DMODEL_DIR}/TerminalBlock_Phoenix.3dshapes/TerminalBlock_Phoenix_MKDS-1,5-2_1x02_P5.00mm_Horizontal.step"
 			(offset
 				(xyz 0 0 0)
@@
 			(layers "*.Cu" "*.Mask")
 			(remove_unused_layers no)
-			(net "Net-(J15-Pin_2)")
+			(net "Selonoid")
 			(pinfunction "~_3")
 			(pintype "passive")
@@
 		)
 		(embedded_fonts no)
+		(model "C:/Users/Lenovo L13/OneDrive/Documents/KiCad/10.0/footprints/IRFZ44N/IRFZ44N.step"
+			(offset
+				(xyz 0 0 -11.5)
+			)
+			(scale
+				(xyz 1 1 1)
+			)
+			(rotate
+				(xyz -90 -0 -0)
+			)
+		)
 	)
 	(footprint "TerminalBlock:TerminalBlock_MaiXu_MX126-5.0-02P_1x02_P5.00mm"
@@
 		(descr "terminal block MaiXu MX126-5.0-02P, 2 pins, pitch 5mm, size 10.5x7.8mm, drill diameter 1.3mm, pad diameter 2.8mm, https://www.lcsc.com/datasheet/lcsc_datasheet_2309150913_MAX-MX126-5-0-03P-GN01-Cu-S-A_C5188435.pdf")
 		(tags "THT terminal block MaiXu MX126-5.0-02P pitch 5mm size 10.5x7.8mm drill 1.3mm pad 2.8mm")
-		(property "Reference" "J5"
+		(property "Reference" "M5"
 			(at 2.25 -5.12 90)
 			(layer "F.SilkS")
@@
 		)
 		(embedded_fonts no)
-		(model "${KICAD10_3DMODEL_DIR}/TerminalBlock.3dshapes/TerminalBlock_MaiXu_MX126-5.0-02P_1x02_P5.00mm.step"
+		(model "${KICAD10_3DMODEL_DIR}/TerminalBlock_Phoenix.3dshapes/TerminalBlock_Phoenix_MKDS-1,5-2_1x02_P5.00mm_Horizontal.step"
 			(offset
 				(xyz 0 0 0)
@@
 		(descr "terminal block MaiXu MX126-5.0-02P, 2 pins, pitch 5mm, size 10.5x7.8mm, drill diameter 1.3mm, pad diameter 2.8mm, https://www.lcsc.com/datasheet/lcsc_datasheet_2309150913_MAX-MX126-5-0-03P-GN01-Cu-S-A_C5188435.pdf")
 		(tags "THT terminal block MaiXu MX126-5.0-02P pitch 5mm size 10.5x7.8mm drill 1.3mm pad 2.8mm")
-		(property "Reference" "J1"
+		(property "Reference" "M1"
 			(at 2.25 -5.12 90)
 			(layer "F.SilkS")
@@
 		)
 		(embedded_fonts no)
-		(model "${KICAD10_3DMODEL_DIR}/TerminalBlock.3dshapes/TerminalBlock_MaiXu_MX126-5.0-02P_1x02_P5.00mm.step"
+		(model "${KICAD10_3DMODEL_DIR}/TerminalBlock_Phoenix.3dshapes/TerminalBlock_Phoenix_MKDS-1,5-2_1x02_P5.00mm_Horizontal.step"
 			(offset
 				(xyz 0 0 0)
@@
 		(width 1.5)
 		(layer "B.Cu")
-		(net "Net-(J16-Pin_1)")
+		(net "FO6")
 	)
 	(segment
@@
 		(width 1.5)
 		(layer "B.Cu")
-		(net "Net-(J16-Pin_1)")
+		(net "FO6")
 	)
 	(segment
@@
 		(width 1.5)
 		(layer "B.Cu")
-		(net "Net-(J16-Pin_1)")
+		(net "FO6")
 	)
 	(segment
@@
 		(width 1.5)
 		(layer "B.Cu")
-		(net "Net-(J16-Pin_1)")
+		(net "FO6")
 	)
 	(segment
@@
 		(width 1.5)
 		(layer "B.Cu")
-		(net "Net-(J16-Pin_1)")
+		(net "FO6")
 	)
 	(segment
@@
 		(width 1.5)
 		(layer "B.Cu")
-		(net "Net-(J16-Pin_1)")
+		(net "FO6")
 	)
 	(segment
@@
 		(width 1.5)
 		(layer "B.Cu")
-		(net "Net-(J16-Pin_1)")
+		(net "FO6")
 	)
 	(segment
@@
 		(width 1.5)
 		(layer "B.Cu")
-		(net "Net-(J16-Pin_1)")
+		(net "FO6")
 	)
 	(segment
@@
 		(width 1.5)
 		(layer "B.Cu")
-		(net "Net-(J16-Pin_1)")
+		(net "FO6")
 	)
 	(segment
@@
 		(width 1.5)
 		(layer "B.Cu")
-		(net "Net-(J16-Pin_2)")
+		(net "BO6")
 	)
 	(segment
@@
 		(width 1.5)
 		(layer "B.Cu")
-		(net "Net-(J16-Pin_2)")
+		(net "BO6")
 	)
 	(segment
@@
 		(width 1.5)
 		(layer "B.Cu")
-		(net "Net-(J16-Pin_2)")
+		(net "BO6")
 	)
 	(segment
@@
 		(width 1.5)
 		(layer "B.Cu")
-		(net "Net-(J16-Pin_2)")
+		(net "BO6")
 	)
 	(segment
@@
 		(width 1.5)
 		(layer "B.Cu")
-		(net "Net-(J16-Pin_2)")
+		(net "BO6")
 	)
 	(segment
@@
 		(width 1.5)
 		(layer "B.Cu")
-		(net "Net-(J16-Pin_2)")
+		(net "BO6")
 	)
 	(segment
@@
 		(width 1.5)
 		(layer "B.Cu")
-		(net "Net-(J16-Pin_2)")
+		(net "BO6")
 	)
 	(segment
@@
 		(width 1.5)
 		(layer "B.Cu")
-		(net "Net-(J16-Pin_2)")
+		(net "BO6")
 	)
 	(segment
@@
 		(width 1.5)
 		(layer "B.Cu")
-		(net "Net-(J16-Pin_2)")
+		(net "BO6")
 	)
 	(segment
@@
 		(width 1.5)
 		(layer "B.Cu")
-		(net "Net-(J16-Pin_2)")
+		(net "BO6")
 	)
 	(segment
@@
 		(width 0.8)
 		(layer "B.Cu")
-		(net "Net-(J15-Pin_2)")
+		(net "Selonoid")
 	)
 	(segment
@@
 		(width 0.8)
 		(layer "B.Cu")
-		(net "Net-(J15-Pin_2)")
+		(net "Selonoid")
 	)
 	(segment
@@
 		(width 0.8)
 		(layer "B.Cu")
-		(net "Net-(J15-Pin_2)")
+		(net "Selonoid")
 	)
 	(segment
@@
 		(width 0.8)
 		(layer "B.Cu")
-		(net "Net-(J15-Pin_2)")
+		(net "Selonoid")
 	)
 	(segment
@@
 		(fill yes
 			(thermal_gap 0.5)
-			(thermal_bridge_width 1)
+			(thermal_bridge_width 1.5)
 			(island_removal_mode 0)
 		)

Commit message: update PCB
Parts:
- removed R6: 0, Resistor_SMD:R_1206_3216Metric_Pad1.30x1.75mm_HandSolder
- moved F7 0.72 mm to (209.5, 73.7)
- moved F6 0.54 mm to (209.6, 55.9)
- renumbered C11 to C0, D6 to D0, F8 to F0, M6 to M0
Connections:
- net BO6 renamed BO0
- net FO6 renamed FO0
- J14 pad 1: P12 -> P11
- J14 pad 2: GND -> P13
- J14 pad 3: Net-(J14-Pad3) -> GND
- J14 pad 4: GND -> P12
- J14 pad 5: P13 -> GND
Routing:
- net Net-(J14-Pad3): track 27.5 -> 0.00 mm
- net P11: track 74.4 -> 94.5 mm
- net P12: track 112.1 -> 98.4 mm
- net +5V b: track 68.6 -> 78.2 mm, vias 3 -> 2
- net P13: track 103.4 -> 96.5 mm
- net P40: track 46.6 -> 44.1 mm
- net Net-(J10-Pin_3): track 24.2 -> 26.1 mm

Commit message: Update PCB
Parts:
- J10: moved to B.Cu
- moved U8 1.69 mm to (226.0, 60.5)
- moved C13 1.59 mm to (232.8, 91.0)
- moved C5 1.59 mm to (183.9, 36.1)
- moved J13 1.59 mm to (221.7, 75.8)
- moved M3 1.59 mm to (162.4, 67.2)
- moved R4 1.59 mm to (237.0, 93.4)
- moved S1 1.59 mm to (245.2, 47.6)
- moved S2 1.59 mm to (245.2, 55.4)
- moved C0 1.59 mm to (183.5, 104.3)
- moved C1 1.59 mm to (184.0, 90.1)
- moved C10 1.59 mm to (237.0, 85.1)
- moved C2 1.59 mm to (183.7, 76.1)
- moved C3 1.59 mm to (184.2, 63.5)
- moved C4 1.59 mm to (183.8, 49.9)
- moved C6 1.59 mm to (218.3, 40.4)
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Connections:
- C9 pad 1: Net-(J10-Pin_3) -> Net-(J10-Pin_4)
- F6 pad 1: Net-(J10-Pin_3) -> Net-(J10-Pin_4)
- F7 pad 1: Net-(J10-Pin_3) -> Net-(J10-Pin_4)
- J10 pad 1: +12V -> GND
- J10 pad 2: GND -> +12V
- J10 pad 3: Net-(J10-Pin_3) -> GND
- J10 pad 4: GND -> Net-(J10-Pin_4)
Routing:
- net Net-(J10-Pin_3): track 26.1 -> 0.00 mm
- net Net-(J10-Pin_4): track 0.00 -> 26.1 mm
