File: MainBoardTrans_Unlimited2026/MainBoardTrans_Unlimited2026.kicad_sch (KiCad schematic)
At the start: 64 parts, among them J10 DSN-MINI-360, J11 pin_H, J12 RST, J13 I2C, J14 RJ45_Shielded, J15 Solenoid, J6 molex, J7 xt30, J8 Tblock, J9 ID-BAT, Q1 IRFZ44N, U1 TA6586, U10 TA6586, U2 TA6586, U3 TA6586, U4 TA6586, U5 TA6586, U6 ESP32-S3-DEVKITC-1, U7 ACS712xLCTR-05B, U8 BNO085, U9 AMS1117-3.3

Commit message: update pcb
Parts:
- renumbered J1 to M1, J2 to M2, J3 to M3, J4 to M4, J5 to M5, J16 to M6
Changed lines of the file:
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@@
 		(dnp no)
 		(fields_autoplaced yes)
-		(property "Reference" "J4"
+		(property "Reference" "M4"
 			(at 54.61 190.4999 0)
 			(show_name no)
@@
 			(project "MainBoardTrans_Unlimited2026"
 				(path "/5d49f12a-b7fe-4d5f-b487-25d02c2ee0eb"
-					(reference "J4")
+					(reference "M4")
 					(unit 1)
 				)
@@
 		(dnp no)
 		(fields_autoplaced yes)
-		(property "Reference" "J16"
+		(property "Reference" "M6"
 			(at 147.32 126.9999 0)
 			(show_name no)
@@
 			(project "MainBoardTrans_Unlimited2026"
 				(path "/5d49f12a-b7fe-4d5f-b487-25d02c2ee0eb"
-					(reference "J16")
+					(reference "M6")
 					(unit 1)
 				)
@@
 		(dnp no)
 		(fields_autoplaced yes)
-		(property "Reference" "J5"
+		(property "Reference" "M5"
 			(at 76.2 180.3399 0)
 			(show_name no)
@@
 			(project "MainBoardTrans_Unlimited2026"
 				(path "/5d49f12a-b7fe-4d5f-b487-25d02c2ee0eb"
-					(reference "J5")
+					(reference "M5")
 					(unit 1)
 				)
@@
 		(dnp no)
 		(fields_autoplaced yes)
-		(property "Reference" "J2"
+		(property "Reference" "M2"
 			(at 34.29 190.4999 0)
 			(show_name no)
@@
 			(project "MainBoardTrans_Unlimited2026"
 				(path "/5d49f12a-b7fe-4d5f-b487-25d02c2ee0eb"
-					(reference "J2")
+					(reference "M2")
 					(unit 1)
 				)
@@
 		(dnp no)
 		(fields_autoplaced yes)
-		(property "Reference" "J1"
+		(property "Reference" "M1"
 			(at 34.29 180.3399 0)
 			(show_name no)
@@
 			(project "MainBoardTrans_Unlimited2026"
 				(path "/5d49f12a-b7fe-4d5f-b487-25d02c2ee0eb"
-					(reference "J1")
+					(reference "M1")
 					(unit 1)
 				)
@@
 		(dnp no)
 		(fields_autoplaced yes)
-		(property "Reference" "J3"
+		(property "Reference" "M3"
 			(at 54.61 180.3399 0)
 			(show_name no)
@@
 			(project "MainBoardTrans_Unlimited2026"
 				(path "/5d49f12a-b7fe-4d5f-b487-25d02c2ee0eb"
-					(reference "J3")
+					(reference "M3")
 					(unit 1)
 				)

Commit message: update PCB
Parts:
- removed R6: 0, Resistor_SMD:R_1206_3216Metric_Pad1.30x1.75mm_HandSolder, symbol Device:R_Small
- renumbered C11 to C0, D6 to D0, F8 to F0, M6 to M0
Connections:
- net GND: now also J14.3, J14.5; no longer J14.2, J14.4
- net P11: now also J14.1
- net P12: now also J14.4; no longer J14.1
- net P13: now also J14.2; no longer J14.5
- net BO6 renamed BO0
- net FO6 renamed FO0

Commit message: Update PCB
Connections:
- net +12V: now also J10.2 (Pin_2); no longer J10.1 (Pin_1)
- net GND: now also J10.1 (Pin_1), J10.3 (Pin_3); no longer J10.2 (Pin_2), J10.4 (Pin_4)
- net at C9.1, F6.1, F7.1: now also J10.4 (Pin_4); no longer J10.3 (Pin_3)
Changed lines of the file:
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@@
 	)
 	(junction
-		(at 171.45 46.99)
+		(at 24.13 20.32)
 		(diameter 0)
 		(color 0 0 0 0)
 	)
 	(junction
-		(at 24.13 20.32)
+		(at 64.77 54.61)
 		(diameter 0)
 		(color 0 0 0 0)
 	)
 	(junction
-		(at 64.77 54.61)
+		(at 29.21 114.3)
 		(diameter 0)
 		(color 0 0 0 0)
 	)
 	(junction
-		(at 29.21 114.3)
+		(at 176.53 48.26)
 		(diameter 0)
 		(color 0 0 0 0)
@@
 	)
 	(junction
+		(at 171.45 44.45)
+		(diameter 0)
+		(color 0 0 0 0)
+	)
+	(junction
 		(at 102.87 157.48)
 		(diameter 0)
@@
 	(wire
 		(pts
-			(xy 64.77 83.82) (xy 64.77 86.36)
+			(xy 172.72 38.1) (xy 172.72 41.91)
 		)
 		(stroke
@@
 	(wire
 		(pts
-			(xy 64.77 118.11) (xy 64.77 120.65)
+			(xy 173.99 40.64) (xy 173.99 46.99)
+		)
+		(stroke
+			(width 0)
+			(type default)
+		)
+	)
+	(wire
+		(pts
+			(xy 64.77 83.82) (xy 64.77 86.36)
 		)
 		(stroke
@@
 	(wire
 		(pts
-			(xy 172.72 44.45) (xy 170.18 44.45)
+			(xy 64.77 118.11) (xy 64.77 120.65)
 		)
 		(stroke
@@
 	(wire
 		(pts
-			(xy 175.26 46.99) (xy 171.45 46.99)
+			(xy 171.45 39.37) (xy 170.18 39.37)
+		)
+		(stroke
+			(width 0)
+			(type default)
+		)
+	)
+	(wire
+		(pts
+			(xy 175.26 45.72) (xy 171.45 45.72)
 		)
 		(stroke
@@
 	(wire
 		(pts
-			(xy 170.18 41.91) (xy 171.45 41.91)
+			(xy 31.75 52.07) (xy 34.29 52.07)
 		)
 		(stroke
@@
 	(wire
 		(pts
-			(xy 31.75 52.07) (xy 34.29 52.07)
+			(xy 97.79 149.86) (xy 102.87 149.86)
 		)
 		(stroke
@@
 	(wire
 		(pts
-			(xy 97.79 149.86) (xy 102.87 149.86)
+			(xy 190.5 66.04) (xy 190.5 68.58)
 		)
 		(stroke
@@
 	(wire
 		(pts
-			(xy 190.5 66.04) (xy 190.5 68.58)
+			(xy 152.4 101.6) (xy 149.86 101.6)
 		)
 		(stroke
@@
 	(wire
 		(pts
-			(xy 152.4 101.6) (xy 149.86 101.6)
+			(xy 31.75 83.82) (xy 34.29 83.82)
 		)
 		(stroke
@@
 	(wire
 		(pts
-			(xy 31.75 83.82) (xy 34.29 83.82)
+			(xy 172.72 41.91) (xy 170.18 41.91)
 		)
 		(stroke
@@
 	(wire
 		(pts
+			(xy 171.45 44.45) (xy 171.45 45.72)
+		)
+		(stroke
+			(width 0)
+			(type default)
+		)
+	)
+	(wire
+		(pts
 			(xy 175.26 77.47) (xy 179.07 77.47)
 		)
@@
 	(wire
 		(pts
-			(xy 172.72 40.64) (xy 172.72 44.45)
-		)
-		(stroke
-			(width 0)
-			(type default)
-		)
-	)
-	(wire
-		(pts
 			(xy 24.13 146.05) (xy 29.21 146.05)
 		)
@@
 	(wire
 		(pts
+			(xy 173.99 46.99) (xy 170.18 46.99)
+		)
+		(stroke
+			(width 0)
+			(type default)
+		)
+	)
+	(wire
+		(pts
 			(xy 247.65 124.46) (xy 247.65 127)
 		)
@@
 	(wire
 		(pts
-			(xy 172.72 40.64) (xy 176.53 40.64)
+			(xy 173.99 40.64) (xy 176.53 40.64)
 		)
 		(stroke
@@
 	(wire
 		(pts
-			(xy 175.26 48.26) (xy 175.26 46.99)
+			(xy 175.26 48.26) (xy 175.26 45.72)
 		)
 		(stroke
@@
 	(wire
 		(pts
-			(xy 171.45 46.99) (xy 170.18 46.99)
-		)
-		(stroke
-			(width 0)
-			(type default)
-		)
-	)
-	(wire
-		(pts
 			(xy 67.31 128.27) (xy 64.77 128.27)
 		)
@@
 	(wire
 		(pts
+			(xy 170.18 44.45) (xy 171.45 44.45)
+		)
+		(stroke
+			(width 0)
+			(type default)
+		)
+	)
+	(wire
+		(pts
 			(xy 31.75 152.4) (xy 31.75 153.67)
 		)
@@
 	(wire
 		(pts
-			(xy 171.45 41.91) (xy 171.45 46.99)
+			(xy 171.45 39.37) (xy 171.45 44.45)
 		)
 		(stroke
@@
 	(symbol
 		(lib_id "power:+12V")
-		(at 170.18 39.37 0)
+		(at 172.72 38.1 0)
 		(unit 1)
 		(body_style 1)
@@
 		(dnp no)
 		(property "Reference" "#PWR019"
-			(at 170.18 43.18 0)
+			(at 172.72 41.91 0)
 			(hide yes)
 			(show_name no)
@@
 		)
 		(property "Value" "+12V"
-			(at 167.64 35.306 0)
+			(at 170.18 34.036 0)
 			(show_name no)
 			(do_not_autoplace no)
@@
 		)
 		(property "Footprint" ""
-			(at 170.18 39.37 0)
+			(at 172.72 38.1 0)
 			(hide yes)
 			(show_name no)
@@
 		)
 		(property "Datasheet" ""
-			(at 170.18 39.37 0)
+			(at 172.72 38.1 0)
 			(hide yes)
 			(show_name no)
@@
 		)
 		(property "Description" "Power symbol creates a global label with name \"+12V\""
-			(at 170.18 39.37 0)
+			(at 172.72 38.1 0)
 			(hide yes)
 			(show_name no)
@@
 	(symbol
 		(lib_id "power:GND")
-		(at 171.45 46.99 0)
+		(at 176.53 48.26 0)
 		(unit 1)
 		(body_style 1)
@@
 		(fields_autoplaced yes)
 		(property "Reference" "#PWR017"
-			(at 171.45 53.34 0)
+			(at 176.53 54.61 0)
 			(hide yes)
 			(show_name no)
@@
 		)
 		(property "Value" "GND"
-			(at 171.45 52.07 0)
+			(at 176.53 53.34 0)
 			(show_name no)
 			(do_not_autoplace no)
@@
 		)
 		(property "Footprint" ""
-			(at 171.45 46.99 0)
+			(at 176.53 48.26 0)
 			(hide yes)
 			(show_name no)
@@
 		)
 		(property "Datasheet" ""
-			(at 171.45 46.99 0)
+			(at 176.53 48.26 0)
 			(hide yes)
 			(show_name no)
@@
 		)
 		(property "Description" "Power symbol creates a global label with name \"GND\" , ground"
-			(at 171.45 46.99 0)
+			(at 176.53 48.26 0)
 			(hide yes)
 			(show_name no)
