File: esp32-cam_holder/esp32-cam_holder.kicad_pcb (KiCad board)
At the start: 2 copper layers, 28 x 55 mm, 6 parts, among them J1 RJ45_Shielded, J2 Conn_01x03_Pin, U1 ESP32-CAM

Commit message: update
Parts:
- J2: value Conn_01x03_Pin -> UART; footprint Connector_PinHeader_2.54mm:PinHeader_1x03_P2.54mm_Horizontal -> Connector_PinHeader_2.54mm:PinHeader_1x04_P2.54mm_Horizontal
- moved J2 23.4 mm to (145.6, 21.7), turned to 90 degrees
- moved G*** 16.1 mm to (151.1, 41.4)
Connections:
- J2 pad 1: RX -> +5V
- J2 pad 3: GND -> RX
Routing:
- net +5V: track 48.5 -> 57.4 mm
- net TX: track 16.8 -> 20.3 mm
