File: MainBoard_Unlimited26/MainBoard_Unlimited26A/MainBoard_Unlimited26A.kicad_pcb (KiCad board)
At the start: 2 copper layers, 95 x 60 mm, 39 parts, among them J1 XT, J2 Screw_Terminal_01x02, J3 BAT, J4 EN, J5 UART, J6 UART, J7 VL5, P1 MP1584, P2 SERVO, Q1 IRFZ44N, U11 ACS712xLCTR-05B, U7 ESP32-DEVKIT-V1, U8 MPU6050/BNO085 I2C, U9 AMS1117-3.3

Commit message: update
Parts:
- moved U8 37.8 mm to (160.3, 111.5)
- moved J7 37.2 mm to (165.3, 111.3)
- moved C8 36.7 mm to (153.5, 110.2)
- moved S5 36.4 mm to (170.5, 78.4)
- moved S4 36.4 mm to (162.7, 78.4)
- moved C9 36.4 mm to (168.3, 65.1)
- moved S3 36.4 mm to (154.9, 78.3)
- moved S2 36.4 mm to (147.1, 78.3)
- moved S1 36.4 mm to (139.5, 78.3)
- moved J2 36.4 mm to (131.4, 65.5)
- moved C11 36.4 mm to (166.3, 87.8)
- moved C12 36.4 mm to (173.7, 106.0)
- moved C6 36.4 mm to (126.8, 97.4)
- moved C7 36.4 mm to (149.8, 95.7)
- moved F6 36.4 mm to (114.0, 92.8)
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Routing:
- net +6V: track 54.6 -> 57.3 mm
- net D19: track 85.4 -> 84.0 mm
- net D18: track 91.9 -> 90.5 mm
- net D26: track 43.8 -> 42.9 mm
- net D33: track 54.8 -> 53.9 mm
- net D23: track 64.4 -> 63.6 mm
Other:
- outline, holes or cut-outs redrawn
