File: MainBoard_Unlimited26/MainBoard_Unlimited26B/MainBoard_Unlimited26B.kicad_sch (KiCad schematic)
At the start: 40 parts, among them J1 power, J2 Conn_01x04_Pin, U1 TA6586, U10 TA6586, U2 TA6586, U3 TA6586, U4 TA6586, U5 TA6586, U6 815

Commit message: update
Parts:
- removed C12: AB conn, Connector_JST:JST_XH_S4B-XH-A-1_1x04_P2.50mm_Horizontal, symbol Connector:Conn_01x04_Pin
- removed J2: Conn_01x04_Pin, Connector_PinHeader_2.54mm:PinHeader_1x04_P2.54mm_Horizontal, symbol Connector:Conn_01x04_Pin
- removed U6: 815, pca:MODULE_815_B, symbol 815:815
- added C11, C12, C6, C7, C8, C9: 0.1uF, Capacitor_SMD:C_0805_2012Metric_Pad1.18x1.45mm_HandSolder, symbol Device:C_Small
- added D13: D_Schottky, Diode_SMD:D_SMA, symbol Device:D_Schottky
- added F6: Polyfuse, Fuse:Fuse_1812_4532Metric, symbol Device:Polyfuse
- added J2: Conn_01x03_Pin, Connector_JST:JST_XH_B3B-XH-A_1x03_P2.50mm_Vertical, symbol Connector:Conn_01x03_Pin
- added U7: ZC323000, STM blue pill:MODULE_ZC323000, symbol ZC323000:ZC323000
- added U8: MP1584_3A_Mini, mp1548:Mini360, symbol MP1584_3A_Mini:MP1584_3A_Mini
- J1: footprint TerminalBlock:TerminalBlock_MaiXu_MX126-5.0-02P_1x02_P5.00mm -> terminal block right angel:TE_282815-2
Connections:
- net +12V: now also J1.1 (Pin_1), D13.2 (A); no longer J1.2 (Pin_2)
- net at C10.1, D11.1 (K), D12.1 (K)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: now also C12.1
- net at C2.1, D2.1 (K), D7.1 (K)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: now also C7.1
- net at C1.1, D1.1 (K), D6.1 (K)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: now also C6.1
- net at F2.2: now also D2.2 (A); no longer D7.2 (A)
- net at C3.1, D3.1 (K), D8.1 (K)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: now also C8.1
- net at F3.2: now also D3.2 (A); no longer D8.2 (A)
- net at C5.1, D10.1 (K), D5.1 (K)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: now also C11.1
- net at F5.2: now also D5.2 (A); no longer D10.2 (A)
- net at F4.2: now also D4.2 (A); no longer D9.2 (A)
- net at C4.1, D4.1 (K), D9.1 (K)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: now also C9.1
- net GND renamed G
- net G: now also D10.2 (A), D7.2 (A), D8.2 (A), D9.2 (A), J1.2 (Pin_2), C11.2, C12.2, C6.2, C7.2, C8.2, C9.2, J2.3 (Pin_3), U7.19 (G), U7.20 (G), U7.39 (G), U8.1 (VIN-), U8.3 (VOUT-); no longer D2.2 (A), D3.2 (A), D4.2 (A), D5.2 (A), J1.1 (Pin_1)
- net PCA1 renamed PB9
- net PB9: now also U7.37 (B9)
- net PCA10 renamed PA7
- net PA7: now also U7.12 (A7)
- net PCA11 renamed PB0
- net PB0: now also U7.13 (B0)
- net PCA12 renamed PB1
- net PB1: now also U7.14 (B1)
- net PCA2 renamed PB8
- net PB8: now also U7.36 (B8)
- net PCA3 renamed PB7
- net PB7: now also U7.35 (B7)
- net PCA4 renamed PB6
- net PB6: now also U7.34 (B6)
- net PCA5 renamed PA11
- net PA11: now also U7.28 (A11)
- net PCA6 renamed PA10
- net PA10: now also U7.27 (A10)
- net PCA7 renamed PA9
- net PA9: now also U7.26 (A9)
- net PCA8 renamed PA8
- net PA8: now also U7.25 (A8)
- net PCA9 renamed PA6
- net PA6: now also U7.11 (A6)
- new net: D13.1 (K), U8.2 (VIN+)
- new net: F6.1, U8.4 (VOUT+)
- new net +5V: F6.2, U7.38 (5V)
- new net 3.3: U7.18 (3.3), U7.40 (3.3)
- new net PA0: U7.5 (A0)
- new net PA1: U7.6 (A1)
- new net RX: J2.2 (Pin_2), U7.8 (A3)
- new net TX: J2.1 (Pin_1), U7.7 (A2)
Other:
- moved on the sheet: C1, C10, D1, D11, D12, D6, F1, F7, J1
